Commit message: Updated head turing limits, suitable for robot without casing.

File: desire_description/ros/urdf/head_v0/head.urdf.xacro (robot description, xacro)
@@ -17,5 +17,5 @@
 			<dynamics damping="0.1" />
 			<calibration rising="${head_pan_ref}" falling="${head_pan_ref}"/>
-			<limit effort="100" lower="-0.7" upper="0.7" velocity="0.5"/>
+			<limit effort="100" lower="-1.4" upper="1.4" velocity="0.5"/>
 		</joint>
 		<link name="${name}_pan_link">
